File: Thermolino2.kicad_pcb (KiCad board)
At the start: 2 copper layers, 50.9 x 53.3 mm, 21 parts, among them J1 Screw_Terminal_01x02, J2 Conn_01x02, J3 Conn_02x08_Odd_Even, U1 MAX31856

Commit message: Added Logo
Parts:
- added G***: LOGO, Thermolino2:Logo, F.Cu at (168.5, 110.9)
Other:
- board text added: "Elchworks"
